Commit message: old g1 removed, new g1 there

File: g1_multiple_pkg_warehouse/environment.urdf (robot description, URDF)
Before this commit: robot environment, 28 links, 27 joints
Links:
- removed link a2edc57a-5c9a-4682-89d5-b6b465b9369e/odom
- added link aba61a87-38cb-438a-ac9f-631cb82ae6f0/odom
Joints:
- removed joint a2edc57a-5c9a-4682-89d5-b6b465b9369e/default_T_odom
- added joint aba61a87-38cb-438a-ac9f-631cb82ae6f0/default_T_odom: type floating, parent default, child aba61a87-38cb-438a-ac9f-631cb82ae6f0/odom, origin xyz=1.75 7.41 0.7923 rpy=0.0 0.0 0.0

File: g1_multiple_pkg_warehouse/unitreeg1.urdf (robot description, URDF)
Before this commit: robot unitreeg1, 57 links, 56 joints
Links:
- removed link parcel
Joints:
- removed joint left_hand_tool_frame_T_parcel
- joint offis_unitree_g1/left_hand_palm_joint: origin xyz=0.0415 0.003 -0.0 rpy=0.0 0.0 0.0 -> xyz=0.0415 0.003 0.0 rpy=0.0 0.0 0.0
- joint offis_unitree_g1/mid360_joint: origin xyz=0.000283 3e-05 0.41618 rpy=-0.0 0.040143 -0.0 -> xyz=0.000284 3e-05 0.41618 rpy=-0.0 0.040143 -0.0
- joint offis_unitree_g1/right_hand_palm_joint: origin xyz=0.0415 -0.003 0.0 rpy=0.0 0.0 0.0 -> xyz=0.0415 -0.003 -0.0 rpy=0.0 0.0 0.0
