Commit message: placement scene: add real living furniture (bookshelf, tv_stand, entrance, dock)
Add four box furniture bodies + a back-wall to apartment.urdf so the living-room
destinations are physically real and reachable, and wire validated performPoses in
scene.json (physical: true). Back-wall behind the furniture forces a west-side
approach (mirrors why the kitchen wall is reliable). Restores the original 5-object
demo (milk, dirty_mug, keys, book, tv_remote) — now 5/5 placed on real furniture,
each within <0.01 m, fresh-process per object (as the viewer runs it).

Co-Authored-By: Claude Opus 4.8 <noreply@anthropic.com>

File: PR2_Apartment_Placement/apartment.urdf (robot description, URDF)
Before this commit: robot apartment, 113 links, 112 joints
Links:
- added link bookshelf; collision box size=0.30 0.50 0.75; visual box size=0.30 0.50 0.75
- added link charging_dock; collision box size=0.25 0.30 0.75; visual box size=0.25 0.30 0.75
- added link entrance_console; collision box size=0.35 0.40 0.80; visual box size=0.35 0.40 0.80
- added link living_backwall; collision box size=0.2 4.0 2.0; visual box size=0.2 4.0 2.0
- added link tv_stand; collision box size=0.35 0.60 0.80; visual box size=0.35 0.60 0.80
Joints:
- added joint bookshelf_joint: type fixed, parent apartment_root, child bookshelf, origin xyz=8.0 3.4 0.0 rpy=0 0 0
- added joint charging_dock_joint: type fixed, parent apartment_root, child charging_dock, origin xyz=8.0 0.5 0.0 rpy=0 0 0
- added joint entrance_console_joint: type fixed, parent apartment_root, child entrance_console, origin xyz=8.0 2.6 0.0 rpy=0 0 0
- added joint living_backwall_joint: type fixed, parent apartment_root, child living_backwall, origin xyz=8.7 2.3 0.0 rpy=0 0 0
- added joint tv_stand_joint: type fixed, parent apartment_root, child tv_stand, origin xyz=8.0 1.8 0.0 rpy=0 0 0
